File: UA-IOTENSR/UA-IOTENSR.sch (KiCad schematic (older format))
At the start: 4 parts

Commit message: Removing rescue libraries
Parts:
- removed J?: S2B-ZR-SM4A-TF(LF)(SN), JST_S2B-ZR-SM4A-TF(LF)(SN), symbol JSTConns:S2B-ZR-SM4A-TF(LF)(SN)
- removed U?: BQ24196RGER, QFN50P400X400X100-25N, symbol TI_PMICs:BQ24196RGER
- U?: symbol Espressif:ESP32 -> UA-IOTENSR-rescue:ESP32-Espressif
Connections:
- wire segments 20 -> 19
Other:
- moved on the sheet: U?
Changed lines of the file:
@@
 $EndDescr
 $Comp
-L Espressif:ESP32 U?
+L UA-IOTENSR-rescue:ESP32-Espressif U?
 U 1 1 6195BA45
 P 2850 2650
@@
 L SCD4X:SCD4X U?
 U 1 1 6195D75D
-P 2650 5750
-F 0 "U?" H 2650 6215 50  0000 C CNN
-F 1 "SCD4X" H 2650 6124 50  0000 C CNN
-F 2 "" H 2650 6200 50  0001 C CNN
-F 3 "" H 2650 6200 50  0001 C CNN
-	1    2650 5750
+P 2400 6050
+F 0 "U?" H 2400 6515 50  0000 C CNN
+F 1 "SCD4X" H 2400 6424 50  0000 C CNN
+F 2 "" H 2400 6500 50  0001 C CNN
+F 3 "" H 2400 6500 50  0001 C CNN
+	1    2400 6050
 	1    0    0    -1
 $EndComp
 Wire Wire Line
-	3100 5650 3250 5650
+	2850 5950 3000 5950
 Wire Wire Line
-	3100 5850 3250 5850
-Text GLabel 3250 5650 2    50   Input ~ 0
+	2850 6150 3000 6150
+Text GLabel 3000 5950 2    50   Input ~ 0
 SCL
 Wire Wire Line
@@
 Text GLabel 4500 2550 2    50   Input ~ 0
 SCL
-Text GLabel 3250 5850 2    50   Input ~ 0
+Text GLabel 3000 6150 2    50   Input ~ 0
 SDA
 Wire Wire Line
@@
 	1    0    0    -1
 $EndComp
-$Comp
-L TI_PMICs:BQ24196RGER U?
-U 1 1 61961F51
-P 9900 1900
-F 0 "U?" H 9900 3070 50  0000 C CNN
-F 1 "BQ24196RGER" H 9900 2979 50  0000 C CNN
-F 2 "QFN50P400X400X100-25N" H 9900 1900 50  0001 L BNN
-F 3 "" H 9900 1900 50  0001 L BNN
-	1    9900 1900
-	1    0    0    -1
-$EndComp
-$Comp
-L power:GND #PWR?
-U 1 1 61965BA6
-P 10600 2800
-F 0 "#PWR?" H 10600 2550 50  0001 C CNN
-F 1 "GND" H 10605 2627 50  0000 C CNN
-F 2 "" H 10600 2800 50  0001 C CNN
-F 3 "" H 10600 2800 50  0001 C CNN
-	1    10600 2800
-	1    0    0    -1
-$EndComp
 Wire Wire Line
-	2550 6200 2550 6250
+	2300 6500 2300 6550
 Wire Wire Line
-	2550 6250 2650 6250
+	2300 6550 2400 6550
 Wire Wire Line
-	2750 6250 2750 6200
+	2500 6550 2500 6500
 Wire Wire Line
-	2650 6200 2650 6250
-Connection ~ 2650 6250
+	2400 6500 2400 6550
+Connection ~ 2400 6550
 Wire Wire Line
-	2650 6250 2750 6250
+	2400 6550 2500 6550
 $Comp
 L power:GND #PWR?
 U 1 1 61967846
-P 2650 6250
-F 0 "#PWR?" H 2650 6000 50  0001 C CNN
-F 1 "GND" H 2655 6077 50  0000 C CNN
-F 2 "" H 2650 6250 50  0001 C CNN
-F 3 "" H 2650 6250 50  0001 C CNN
-	1    2650 6250
+P 2400 6550
+F 0 "#PWR?" H 2400 6300 50  0001 C CNN
+F 1 "GND" H 2405 6377 50  0000 C CNN
+F 2 "" H 2400 6550 50  0001 C CNN
+F 3 "" H 2400 6550 50  0001 C CNN
+	1    2400 6550
 	1    0    0    -1
 $EndComp
-Wire Wire Line
-	10600 1000 10750 1000
-Text GLabel 10750 1000 2    50   Input ~ 0
-BATT
 Wire Wire Line
 	8750 3650 9150 3650
@@
 	9350 3800 9500 3800
 Connection ~ 9350 4000
-$Comp
-L JSTConns:S2B-ZR-SM4A-TF(LF)(SN) J?
-U 1 1 6196E09B
-P 9900 3900
-F 0 "J?" H 10128 3996 50  0000 L CNN
-F 1 "S2B-ZR-SM4A-TF(LF)(SN)" H 10128 3905 50  0000 L CNN
-F 2 "JST_S2B-ZR-SM4A-TF(LF)(SN)" H 9900 3900 50  0001 L BNN
-F 3 "" H 9900 3900 50  0001 L BNN
-F 4 "Manufacturer Recommendations" H 9900 3900 50  0001 L BNN "STANDARD"
-F 5 "JST" H 9900 3900 50  0001 L BNN "MF"
-F 6 "N/A" H 9900 3900 50  0001 L BNN "PARTREV"
-	1    9900 3900
-	1    0    0    -1
-$EndComp
 Wire Wire Line
 	9150 3650 9500 3650

Commit message: Adding correct libraries and removing previous Power System design
Parts:
- removed U?: ESP32, symbol UA-IOTENSR-rescue:ESP32-Espressif
- added U?: ESP32-S3-WROOM-1, Espressif:ESP32-S3-WROOM-1, symbol Espressif:ESP32-S3-WROOM-1
Connections:
- net labels removed: BATT
- wire segments 19 -> 14
Other:
- moved on the sheet: U?
Changed lines of the file:
@@
 $EndDescr
-$Comp
-L UA-IOTENSR-rescue:ESP32-Espressif U?
-U 1 1 6195BA45
-P 2850 2650
-F 0 "U?" H 2875 4465 50  0000 C CNN
-F 1 "ESP32" H 2875 4374 50  0000 C CNN
-F 2 "" H 3100 2900 50  0001 C CNN
-F 3 "https://www.espressif.com/sites/default/files/documentation/esp32_datasheet_en.pdf" H 3100 2900 50  0001 C CNN
-	1    2850 2650
-	1    0    0    -1
-$EndComp
 $Comp
 L SCD4X:SCD4X U?
 U 1 1 6195D75D
-P 2400 6050
-F 0 "U?" H 2400 6515 50  0000 C CNN
-F 1 "SCD4X" H 2400 6424 50  0000 C CNN
-F 2 "" H 2400 6500 50  0001 C CNN
-F 3 "" H 2400 6500 50  0001 C CNN
-	1    2400 6050
+P 1650 5150
+F 0 "U?" H 1650 5615 50  0000 C CNN
+F 1 "SCD4X" H 1650 5524 50  0000 C CNN
+F 2 "" H 1650 5600 50  0001 C CNN
+F 3 "" H 1650 5600 50  0001 C CNN
+	1    1650 5150
 	1    0    0    -1
 $EndComp
 Wire Wire Line
-	2850 5950 3000 5950
+	2100 5050 2250 5050
 Wire Wire Line
-	2850 6150 3000 6150
-Text GLabel 3000 5950 2    50   Input ~ 0
+	2100 5250 2250 5250
+Text GLabel 2250 5050 2    50   Input ~ 0
 SCL
 Wire Wire Line
-	4350 2550 4500 2550
-Text GLabel 4500 2550 2    50   Input ~ 0
+	5650 1550 5800 1550
+Text GLabel 5800 1550 2    50   Input ~ 0
 SCL
-Text GLabel 3000 6150 2    50   Input ~ 0
+Text GLabel 2250 5250 2    50   Input ~ 0
 SDA
 Wire Wire Line
-	4350 2450 4500 2450
-Text GLabel 4500 2450 2    50   Input ~ 0
+	5650 1450 5800 1450
+Text GLabel 5800 1450 2    50   Input ~ 0
 SDA
 $Comp
 L power:GND #PWR?
 U 1 1 61961638
-P 4350 4150
-F 0 "#PWR?" H 4350 3900 50  0001 C CNN
-F 1 "GND" H 4355 3977 50  0000 C CNN
-F 2 "" H 4350 4150 50  0001 C CNN
-F 3 "" H 4350 4150 50  0001 C CNN
-	1    4350 4150
+P 5800 3300
+F 0 "#PWR?" H 5800 3050 50  0001 C CNN
+F 1 "GND" H 5805 3127 50  0000 C CNN
+F 2 "" H 5800 3300 50  0001 C CNN
+F 3 "" H 5800 3300 50  0001 C CNN
+	1    5800 3300
 	1    0    0    -1
 $EndComp
 Wire Wire Line
-	2300 6500 2300 6550
+	1550 5600 1550 5650
 Wire Wire Line
-	2300 6550 2400 6550
+	1550 5650 1650 5650
 Wire Wire Line
-	2500 6550 2500 6500
+	1750 5650 1750 5600
 Wire Wire Line
-	2400 6500 2400 6550
-Connection ~ 2400 6550
+	1650 5600 1650 5650
+Connection ~ 1650 5650
 Wire Wire Line
-	2400 6550 2500 6550
+	1650 5650 1750 5650
 $Comp
 L power:GND #PWR?
 U 1 1 61967846
-P 2400 6550
-F 0 "#PWR?" H 2400 6300 50  0001 C CNN
-F 1 "GND" H 2405 6377 50  0000 C CNN
-F 2 "" H 2400 6550 50  0001 C CNN
-F 3 "" H 2400 6550 50  0001 C CNN
-	1    2400 6550
+P 1650 5650
+F 0 "#PWR?" H 1650 5400 50  0001 C CNN
+F 1 "GND" H 1655 5477 50  0000 C CNN
+F 2 "" H 1650 5650 50  0001 C CNN
+F 3 "" H 1650 5650 50  0001 C CNN
+	1    1650 5650
+	1    0    0    -1
+$EndComp
+$Comp
+L Espressif:ESP32-S3-WROOM-1 U?
+U 1 1 619A01D1
+P 3350 2000
+F 0 "U?" H 3325 3515 50  0000 C CNN
+F 1 "ESP32-S3-WROOM-1" H 3325 3424 50  0000 C CNN
+F 2 "Espressif:ESP32-S3-WROOM-1" H 3350 450 50  0001 C CNN
+F 3 "" H 3350 2300 50  0001 C CNN
+	1    3350 2000
 	1    0    0    -1
 $EndComp
 Wire Wire Line
-	8750 3650 9150 3650
+	5650 3100 5800 3100
 Wire Wire Line
-	9350 4000 9350 4100
+	5800 3100 5800 3200
 Wire Wire Line
-	9350 4100 9150 4100
+	5650 3200 5800 3200
+Connection ~ 5800 3200
 Wire Wire Line
-	9150 4100 9150 4000
+	5800 3200 5800 3300
 Wire Wire Line
-	9150 3650 9150 3750
-$Comp
-L power:GND #PWR?
-U 1 1 6196C16A
-P 9350 4100
-F 0 "#PWR?" H 9350 3850 50  0001 C CNN
-F 1 "GND" H 9355 3927 50  0000 C CNN
-F 2 "" H 9350 4100 50  0001 C CNN
-F 3 "" H 9350 4100 50  0001 C CNN
-	1    9350 4100
-	1    0    0    -1
-$EndComp
-Connection ~ 9350 4100
-Text GLabel 8750 3650 0    50   Input ~ 0
-BATT
-Wire Wire Line
-	9350 4000 9500 4000
-Wire Wire Line
-	9350 4000 9350 3800
-Wire Wire Line
-	9350 3800 9500 3800
-Connection ~ 9350 4000
-Wire Wire Line
-	9150 3650 9500 3650
-Wire Wire Line
-	9500 3650 9500 3700
-Connection ~ 9150 3650
+	5650 3300 5800 3300
+Connection ~ 5800 3300
 $EndSCHEMATC

Commit message: Libraries with more work done on Schem.
Parts:
- added U?: BQ24196RGER, QFN50P400X400X100-25N, symbol PMIC:BQ24196RGER
- added U?: BD33KA5FP-E2, TO252-3_ROM, symbol VoltReg:BD33KA5FP-E2
Connections:
- wire segments 14 -> 15
Other:
- moved on the sheet: U?
Changed lines of the file:
@@
 L SCD4X:SCD4X U?
 U 1 1 6195D75D
-P 1650 5150
-F 0 "U?" H 1650 5615 50  0000 C CNN
-F 1 "SCD4X" H 1650 5524 50  0000 C CNN
-F 2 "" H 1650 5600 50  0001 C CNN
-F 3 "" H 1650 5600 50  0001 C CNN
-	1    1650 5150
+P 9000 2200
+F 0 "U?" H 9000 2665 50  0000 C CNN
+F 1 "SCD4X" H 9000 2574 50  0000 C CNN
+F 2 "" H 9000 2650 50  0001 C CNN
+F 3 "" H 9000 2650 50  0001 C CNN
+	1    9000 2200
 	1    0    0    -1
 $EndComp
 Wire Wire Line
-	2100 5050 2250 5050
+	9450 2100 9600 2100
 Wire Wire Line
-	2100 5250 2250 5250
-Text GLabel 2250 5050 2    50   Input ~ 0
+	9450 2300 9600 2300
+Text GLabel 9600 2100 2    50   Input ~ 0
 SCL
 Wire Wire Line
-	5650 1550 5800 1550
-Text GLabel 5800 1550 2    50   Input ~ 0
+	5750 1700 5900 1700
+Text GLabel 5900 1700 2    50   Input ~ 0
 SCL
-Text GLabel 2250 5250 2    50   Input ~ 0
+Text GLabel 9600 2300 2    50   Input ~ 0
 SDA
 Wire Wire Line
-	5650 1450 5800 1450
-Text GLabel 5800 1450 2    50   Input ~ 0
+	5750 1600 5900 1600
+Text GLabel 5900 1600 2    50   Input ~ 0
 SDA
 $Comp
 L power:GND #PWR?
 U 1 1 61961638
-P 5800 3300
-F 0 "#PWR?" H 5800 3050 50  0001 C CNN
-F 1 "GND" H 5805 3127 50  0000 C CNN
-F 2 "" H 5800 3300 50  0001 C CNN
-F 3 "" H 5800 3300 50  0001 C CNN
-	1    5800 3300
+P 5850 3450
+F 0 "#PWR?" H 5850 3200 50  0001 C CNN
+F 1 "GND" H 5855 3277 50  0000 C CNN
+F 2 "" H 5850 3450 50  0001 C CNN
+F 3 "" H 5850 3450 50  0001 C CNN
+	1    5850 3450
 	1    0    0    -1
 $EndComp
 Wire Wire Line
-	1550 5600 1550 5650
+	8900 2650 8900 2700
 Wire Wire Line
-	1550 5650 1650 5650
+	8900 2700 9000 2700
 Wire Wire Line
-	1750 5650 1750 5600
+	9100 2700 9100 2650
 Wire Wire Line
-	1650 5600 1650 5650
-Connection ~ 1650 5650
+	9000 2650 9000 2700
+Connection ~ 9000 2700
 Wire Wire Line
-	1650 5650 1750 5650
+	9000 2700 9100 2700
 $Comp
 L power:GND #PWR?
 U 1 1 61967846
-P 1650 5650
-F 0 "#PWR?" H 1650 5400 50  0001 C CNN
-F 1 "GND" H 1655 5477 50  0000 C CNN
-F 2 "" H 1650 5650 50  0001 C CNN
-F 3 "" H 1650 5650 50  0001 C CNN
-	1    1650 5650
+P 9000 2700
+F 0 "#PWR?" H 9000 2450 50  0001 C CNN
+F 1 "GND" H 9005 2527 50  0000 C CNN
+F 2 "" H 9000 2700 50  0001 C CNN
+F 3 "" H 9000 2700 50  0001 C CNN
+	1    9000 2700
 	1    0    0    -1
 $EndComp
@@
 L Espressif:ESP32-S3-WROOM-1 U?
 U 1 1 619A01D1
-P 3350 2000
-F 0 "U?" H 3325 3515 50  0000 C CNN
-F 1 "ESP32-S3-WROOM-1" H 3325 3424 50  0000 C CNN
-F 2 "Espressif:ESP32-S3-WROOM-1" H 3350 450 50  0001 C CNN
-F 3 "" H 3350 2300 50  0001 C CNN
-	1    3350 2000
+P 3450 2150
+F 0 "U?" H 3425 3665 50  0000 C CNN
+F 1 "ESP32-S3-WROOM-1" H 3425 3574 50  0000 C CNN
+F 2 "Espressif:ESP32-S3-WROOM-1" H 3450 600 50  0001 C CNN
+F 3 "" H 3450 2450 50  0001 C CNN
+	1    3450 2150
 	1    0    0    -1
 $EndComp
 Wire Wire Line
-	5650 3100 5800 3100
+	5850 3250 5850 3350
 Wire Wire Line
-	5800 3100 5800 3200
+	5750 3250 5850 3250
 Wire Wire Line
-	5650 3200 5800 3200
-Connection ~ 5800 3200
+	5750 3350 5850 3350
+Connection ~ 5850 3350
 Wire Wire Line
-	5800 3200 5800 3300
+	5850 3350 5850 3450
 Wire Wire Line
-	5650 3300 5800 3300
-Connection ~ 5800 3300
+	5750 3450 5850 3450
+Connection ~ 5850 3450
+$Comp
+L PMIC:BQ24196RGER U?
+U 1 1 619B6CD5
+P 1700 6600
+F 0 "U?" H 1700 7770 50  0000 C CNN
+F 1 "BQ24196RGER" H 1700 7679 50  0000 C CNN
+F 2 "QFN50P400X400X100-25N" H 1700 6600 50  0001 L BNN
+F 3 "" H 1700 6600 50  0001 L BNN
+	1    1700 6600
+	1    0    0    -1
+$EndComp
+Wire Wire Line
+	2400 5700 2650 5700
+$Comp
+L VoltReg:BD33KA5FP-E2 U?
+U 1 1 619CA410
+P 2400 5000
+F 0 "U?" H 3200 5387 60  0000 C CNN
+F 1 "BD33KA5FP-E2" H 3200 5281 60  0000 C CNN
+F 2 "TO252-3_ROM" H 3200 5240 60  0001 C CNN
+F 3 "" H 2400 5000 60  0000 C CNN
+	1    2400 5000
+	1    0    0    -1
+$EndComp
 $EndSCHEMATC

Commit message: Adding power system page, reorganizing libraries (more work needed)
Parts:
- removed U?: ESP32-S3-WROOM-1, Espressif:ESP32-S3-WROOM-1, symbol Espressif:ESP32-S3-WROOM-1
- removed U?: BQ24196RGER, QFN50P400X400X100-25N, symbol PMIC:BQ24196RGER
- removed U?: BD33KA5FP-E2, TO252-3_ROM, symbol VoltReg:BD33KA5FP-E2
- added DS101: HDSP-4832, DIPS762W61P254L2540H635Q20N, symbol Samacs:HDSP-4832
- added IC101: LM3914VX_NOPB, PLCC127P990X990X457-20N, symbol Samacs:LM3914VX_NOPB
- added SW101: SW_MEC_5G, symbol Switch:SW_MEC_5G
- added U101: ESP32-S2-WROOM, Espressif:ESP32-S2-WROOM, symbol Espressif:ESP32-S2-WROOM
- gave numbers to parts that had none: 1
Connections:
- net labels added: D+, D-, OTG, VDD
- wire segments 15 -> 24
Other:
- moved on the sheet: U102
Changed lines of the file:
@@
 $Descr A4 11693 8268
 encoding utf-8
-Sheet 1 1
+Sheet 1 2
 Title ""
 Date ""
@@
 $EndDescr
 $Comp
-L SCD4X:SCD4X U?
+L SCD4X:SCD4X U102
 U 1 1 6195D75D
-P 9000 2200
-F 0 "U?" H 9000 2665 50  0000 C CNN
-F 1 "SCD4X" H 9000 2574 50  0000 C CNN
-F 2 "" H 9000 2650 50  0001 C CNN
-F 3 "" H 9000 2650 50  0001 C CNN
-	1    9000 2200
+P 7300 1950
+F 0 "U102" H 7300 2415 50  0000 C CNN
+F 1 "SCD4X" H 7300 2324 50  0000 C CNN
+F 2 "" H 7300 2400 50  0001 C CNN
+F 3 "" H 7300 2400 50  0001 C CNN
+	1    7300 1950
 	1    0    0    -1
 $EndComp
 Wire Wire Line
-	9450 2100 9600 2100
+	7750 1850 7900 1850
 Wire Wire Line
-	9450 2300 9600 2300
-Text GLabel 9600 2100 2    50   Input ~ 0
+	7750 2050 7900 2050
+Text GLabel 7900 1850 2    50   Input ~ 0
 SCL
-Wire Wire Line
-	5750 1700 5900 1700
-Text GLabel 5900 1700 2    50   Input ~ 0
-SCL
-Text GLabel 9600 2300 2    50   Input ~ 0
-SDA
-Wire Wire Line
-	5750 1600 5900 1600
-Text GLabel 5900 1600 2    50   Input ~ 0
+Text GLabel 7900 2050 2    50   Input ~ 0
 SDA
 $Comp
-L power:GND #PWR?
+L power:GND #PWR0101
 U 1 1 61961638
-P 5850 3450
-F 0 "#PWR?" H 5850 3200 50  0001 C CNN
-F 1 "GND" H 5855 3277 50  0000 C CNN
-F 2 "" H 5850 3450 50  0001 C CNN
-F 3 "" H 5850 3450 50  0001 C CNN
-	1    5850 3450
+P 1000 4200
+F 0 "#PWR0101" H 1000 3950 50  0001 C CNN
+F 1 "GND" H 1005 4027 50  0000 C CNN
+F 2 "" H 1000 4200 50  0001 C CNN
+F 3 "" H 1000 4200 50  0001 C CNN
+	1    1000 4200
 	1    0    0    -1
 $EndComp
 Wire Wire Line
-	8900 2650 8900 2700
+	7200 2400 7200 2450
 Wire Wire Line
-	8900 2700 9000 2700
+	7200 2450 7300 2450
 Wire Wire Line
-	9100 2700 9100 2650
+	7400 2450 7400 2400
 Wire Wire Line
-	9000 2650 9000 2700
-Connection ~ 9000 2700
+	7300 2400 7300 2450
+Connection ~ 7300 2450
 Wire Wire Line
-	9000 2700 9100 2700
+	7300 2450 7400 2450
 $Comp
-L power:GND #PWR?
+L power:GND #PWR0104
 U 1 1 61967846
-P 9000 2700
-F 0 "#PWR?" H 9000 2450 50  0001 C CNN
-F 1 "GND" H 9005 2527 50  0000 C CNN
-F 2 "" H 9000 2700 50  0001 C CNN
-F 3 "" H 9000 2700 50  0001 C CNN
-	1    9000 2700
+P 7300 2450
+F 0 "#PWR0104" H 7300 2200 50  0001 C CNN
+F 1 "GND" H 7305 2277 50  0000 C CNN
+F 2 "" H 7300 2450 50  0001 C CNN
+F 3 "" H 7300 2450 50  0001 C CNN
+	1    7300 2450
+	1    0    0    -1
+$EndComp
+Wire Wire Line
+	1000 4000 1100 4000
+Wire Wire Line
+	1000 4100 1100 4100
+Wire Wire Line
+	1000 4200 1100 4200
+$Comp
+L Espressif:ESP32-S2-WROOM U101
+U 1 1 619E5D94
+P 2500 2550
+F 0 "U101" H 2525 4465 50  0000 C CNN
+F 1 "ESP32-S2-WROOM" H 2525 4374 50  0000 C CNN
+F 2 "Espressif:ESP32-S2-WROOM" H 2500 650 50  0001 C CNN
+F 3 "https://www.espressif.com/sites/default/files/documentation/esp32-s2-wroom_esp32-s2-wroom-i_datasheet_en.pdf" H 2500 2550 50  0001 C CNN
+	1    2500 2550
+	1    0    0    -1
+$EndComp
+Wire Wire Line
+	1100 3900 1000 3900
+Wire Wire Line
+	1000 3900 1000 4000
+Connection ~ 1000 4000
+Wire Wire Line
+	1000 4000 1000 4100
+Connection ~ 1000 4100
+Wire Wire Line
+	1000 4100 1000 4200
+Connection ~ 1000 4200
+Wire Wire Line
+	3950 1750 4100 1750
+Text GLabel 4100 1750 2    50   Input ~ 0
+SCL
+Text GLabel 4100 1650 2    50   Input ~ 0
+SDA
+Wire Wire Line
+	3950 1650 4100 1650
+Wire Wire Line
+	4450 1250 4600 1250
+$Comp
+L Switch:SW_MEC_5G SW101
+U 1 1 619D98CD
+P 4250 1250
+F 0 "SW101" H 4250 1535 50  0000 C CNN
+F 1 "SW_MEC_5G" H 4250 1444 50  0000 C CNN
+F 2 "" H 4250 1450 50  0001 C CNN
+F 3 "http://www.apem.com/int/index.php?controller=attachment&id_attachment=488" H 4250 1450 50  0001 C CNN
+	1    4250 1250
+	1    0    0    -1
+$EndComp
+Wire Wire Line
+	3950 1250 4050 1250
+$Comp
+L power:GND #PWR0102
+U 1 1 61A04BEB
+P 4600 1250
+F 0 "#PWR0102" H 4600 1000 50  0001 C CNN
+F 1 "GND" H 4605 1077 50  0000 C CNN
+F 2 "" H 4600 1250 50  0001 C CNN
+F 3 "" H 4600 1250 50  0001 C CNN
+	1    4600 1250
+	1    0    0    -1
+$EndComp
+Wire Wire Line
+	1100 3650 1000 3650
+Text GLabel 1000 3650 0    50   Input ~ 0
+VDD
+Wire Wire Line
+	6850 1900 6650 1900
+Text GLabel 6650 1900 0    50   Input ~ 0
+VDD
+Text GLabel 4100 2550 2    50   Input ~ 0
+D+
+Wire Wire Line
+	3950 2550 4100 2550
+Text GLabel 4100 2650 2    50   Input ~ 0
+D-
+Wire Wire Line
+	3950 2650 4100 2650
+Wire Wire Line
+	6850 2000 6850 1900
+Connection ~ 6850 1900
+Wire Wire Line
+	3950 2350 4100 2350
+Text GLabel 4100 2350 2    50   Input ~ 0
+OTG
+$Comp
+L Samacs:HDSP-4832 DS101
+U 1 1 619CEE0B
+P 9050 4200
+F 0 "DS101" H 9850 4465 50  0000 C CNN
+F 1 "HDSP-4832" H 9850 4374 50  0000 C CNN
+F 2 "DIPS762W61P254L2540H635Q20N" H 10500 4300 50  0001 L CNN
+F 3 "https://datasheet.datasheetarchive.com/originals/distributors/Datasheets-6/DSA-115790.pdf" H 10500 4200 50  0001 L CNN
+F 4 "Avago Light Bar Array Green/Red/Yellow LED Display, 1900 (Green) ??cd, 1900 (Yellow) ??cd, 3500 (Red) ??cd" H 10500 4100 50  0001 L CNN "Description"
+F 5 "6.35" H 10500 4000 50  0001 L CNN "Height"
+F 6 "630-HDSP-4832" H 10500 3900 50  0001 L CNN "Mouser Part Number"
+F 7 "https://www.mouser.co.uk/ProductDetail/Broadcom-Avago/HDSP-4832?qs=pQfy5%252BKCabLkjNEFwaYNQw%3D%3D" H 10500 3800 50  0001 L CNN "Mouser Price/Stock"
+F 8 "Avago Technologies" H 10500 3700 50  0001 L CNN "Manufacturer_Name"
+F 9 "HDSP-4832" H 10500 3600 50  0001 L CNN "Manufacturer_Part_Number"
+	1    9050 4200
 	1    0    0    -1
 $EndComp
 $Comp
-L Espressif:ESP32-S3-WROOM-1 U?
-U 1 1 619A01D1
-P 3450 2150
-F 0 "U?" H 3425 3665 50  0000 C CNN
-F 1 "ESP32-S3-WROOM-1" H 3425 3574 50  0000 C CNN
-F 2 "Espressif:ESP32-S3-WROOM-1" H 3450 600 50  0001 C CNN
-F 3 "" H 3450 2450 50  0001 C CNN
-	1    3450 2150
+L Samacs:LM3914VX_NOPB IC101
+U 1 1 619D4939
+P 5650 4550
+F 0 "IC101" H 7694 4246 50  0000 L CNN
+F 1 "LM3914VX_NOPB" H 7694 4155 50  0000 L CNN
+F 2 "PLCC127P990X990X457-20N" H 7500 5050 50  0001 L CNN
+F 3 "http://www.ti.com/lit/gpn/lm3914" H 7500 4950 50  0001 L CNN
+F 4 "Dot/Bar Display Driver" H 7500 4850 50  0001 L CNN "Description"
+F 5 "4.57" H 7500 4750 50  0001 L CNN "Height"
+F 6 "926-LM3914VX/NOPB" H 7500 4650 50  0001 L CNN "Mouser Part Number"
+F 7 "https://www.mouser.co.uk/ProductDetail/Texas-Instruments/LM3914VX-NOPB?qs=QbsRYf82W3FGYq5LQoAqbA%3D%3D" H 7500 4550 50  0001 L CNN "Mouser Price/Stock"
+F 8 "Texas Instruments" H 7500 4450 50  0001 L CNN "Manufacturer_Name"
+F 9 "LM3914VX/NOPB" H 7500 4350 50  0001 L CNN "Manufacturer_Part_Number"
+	1    5650 4550
 	1    0    0    -1
 $EndComp
-Wire Wire Line
-	5850 3250 5850 3350
-Wire Wire Line
-	5750 3250 5850 3250
-Wire Wire Line
-	5750 3350 5850 3350
-Connection ~ 5850 3350
-Wire Wire Line
-	5850 3350 5850 3450
-Wire Wire Line
-	5750 3450 5850 3450
-Connection ~ 5850 3450
-$Comp
-L PMIC:BQ24196RGER U?
-U 1 1 619B6CD5
-P 1700 6600
-F 0 "U?" H 1700 7770 50  0000 C CNN
-F 1 "BQ24196RGER" H 1700 7679 50  0000 C CNN
-F 2 "QFN50P400X400X100-25N" H 1700 6600 50  0001 L BNN
-F 3 "" H 1700 6600 50  0001 L BNN
-	1    1700 6600
-	1    0    0    -1
-$EndComp
-Wire Wire Line
-	2400 5700 2650 5700
-$Comp
-L VoltReg:BD33KA5FP-E2 U?
-U 1 1 619CA410
-P 2400 5000
-F 0 "U?" H 3200 5387 60  0000 C CNN
-F 1 "BD33KA5FP-E2" H 3200 5281 60  0000 C CNN
-F 2 "TO252-3_ROM" H 3200 5240 60  0001 C CNN
-F 3 "" H 2400 5000 60  0000 C CNN
-	1    2400 5000
-	1    0    0    -1
-$EndComp
+$Sheet
+S 9600 600  1450 650
+U 61A2F8E2
+F0 "Power" 50
+F1 "Power.sch" 50
+$EndSheet
 $EndSCHEMATC
