File: UA-IOTENSR/UA-IOTENSR.sch (KiCad schematic (older format))
At the start: 3 parts, among them J1 Conn_01x04_Male, SW1 SW_DPST, U1 ESP32-S3-MINI-1

Commit message: removed dc+-, ground pour, M3 mounting holes
Parts:
- removed SW1: SW_DPST, SamacSys_Parts:PB400EEQR1BLK, symbol Switch:SW_DPST
- added R1: 10k, SamacSys_Parts:RESC5025X70N, symbol Device:R_US
- added SW1: SW_Push, Button_Switch_THT:SW_Tactile_SPST_Angled_PTS645Vx58-2LFS, symbol Switch:SW_Push
Connections:
- net labels added: PUSHBUTTON
- net labels removed: D+, D-
- wire segments 35 -> 29
- no-connect marks 34 -> 36
Other:
- note added: "PUSHBUTTON"
Changed lines of the file:
@@
 Wire Wire Line
 	1700 3450 1550 3450
-Text GLabel 6500 1400 2    50   Input ~ 0
-D+
-Wire Wire Line
-	6350 1400 6500 1400
-Text GLabel 6500 1500 2    50   Input ~ 0
-D-
-Wire Wire Line
-	6350 1500 6500 1500
 $Sheet
 S 1800 4550 1450 650
@@
 SCD-41 Header
 Wire Wire Line
-	7000 2450 7100 2450
-Wire Wire Line
-	6350 2150 7000 2150
-Wire Wire Line
 	6350 3600 6500 3600
 Wire Wire Line
@@
 NoConn ~ 1700 1500
 NoConn ~ 1700 1750
-NoConn ~ 1700 1850
+NoConn ~ 6350 2150
 NoConn ~ 1700 1950
 NoConn ~ 1700 2050
@@
 	1250 1600 1500 1600
 Connection ~ 1500 1600
-$Comp
-L Switch:SW_DPST SW1
-U 1 1 620C5E9D
-P 7300 2450
-F 0 "SW1" H 7300 2775 50  0000 C CNN
-F 1 "SW_DPST" H 7300 2684 50  0000 C CNN
-F 2 "SamacSys_Parts:PB400EEQR1BLK" H 7300 2450 50  0001 C CNN
-F 3 "~" H 7300 2450 50  0001 C CNN
-	1    7300 2450
-	1    0    0    -1
-$EndComp
-Wire Wire Line
-	7100 2550 7100 2450
-Wire Wire Line
-	7500 2550 7500 2450
-Wire Wire Line
-	7500 2450 7650 2450
-Wire Wire Line
-	7650 2450 7650 2550
-Connection ~ 7500 2450
-Wire Wire Line
-	7500 2450 7500 2350
-Connection ~ 7100 2450
-Wire Wire Line
-	7100 2450 7100 2350
-Wire Wire Line
-	7000 2150 7000 2450
+Wire Wire Line
+	9700 3650 9700 3750
 $Comp
 L power:GND #PWR03
 U 1 1 620D10AA
-P 7650 2550
-F 0 "#PWR03" H 7650 2300 50  0001 C CNN
-F 1 "GND" H 7655 2377 50  0000 C CNN
-F 2 "" H 7650 2550 50  0001 C CNN
-F 3 "" H 7650 2550 50  0001 C CNN
-	1    7650 2550
+P 9700 3750
+F 0 "#PWR03" H 9700 3500 50  0001 C CNN
+F 1 "GND" H 9705 3577 50  0000 C CNN
+F 2 "" H 9700 3750 50  0001 C CNN
+F 3 "" H 9700 3750 50  0001 C CNN
+	1    9700 3750
 	1    0    0    -1
 $EndComp
@@
 Wire Notes Line
 	8300 1400 8300 2400
+Wire Wire Line
+	1700 1850 950  1850
+Text GLabel 950  1850 1    50   Input ~ 0
+PUSHBUTTON
+Text GLabel 8500 3250 0    50   Input ~ 0
+PUSHBUTTON
+$Comp
+L Switch:SW_Push SW1
+U 1 1 624DC38E
+P 9100 3250
+F 0 "SW1" H 9100 3535 50  0000 C CNN
+F 1 "SW_Push" H 9100 3444 50  0000 C CNN
+F 2 "Button_Switch_THT:SW_Tactile_SPST_Angled_PTS645Vx58-2LFS" H 9100 3450 50  0001 C CNN
+F 3 "~" H 9100 3450 50  0001 C CNN
+	1    9100 3250
+	1    0    0    -1
+$EndComp
+Wire Wire Line
+	8500 3250 8900 3250
+Wire Wire Line
+	9300 3250 9700 3250
+Wire Wire Line
+	9700 3250 9700 3350
+$Comp
+L Device:R_US R1
+U 1 1 624E061B
+P 9700 3500
+F 0 "R1" H 9768 3546 50  0000 L CNN
+F 1 "10k" H 9768 3455 50  0000 L CNN
+F 2 "SamacSys_Parts:RESC5025X70N" V 9740 3490 50  0001 C CNN
+F 3 "~" H 9700 3500 50  0001 C CNN
+	1    9700 3500
+	1    0    0    -1
+$EndComp
+Wire Notes Line
+	7900 2850 10000 2850
+Wire Notes Line
+	10000 2850 10000 4000
+Wire Notes Line
+	10000 4000 7900 4000
+Wire Notes Line
+	7900 4000 7900 2850
+Text Notes 7950 3950 0    118  ~ 0
+PUSHBUTTON
+NoConn ~ 6350 1400
+NoConn ~ 6350 1500
 $EndSCHEMATC

Commit message: Zettai Ryouiki
Parts:
- removed R1: 10k, SamacSys_Parts:RESC5025X70N, symbol Device:R_US
- added J3: Conn_01x04_Male, Connector_PinSocket_2.54mm:PinSocket_1x04_P2.54mm_Vertical, symbol Connector:Conn_01x04_Male
Connections:
- wire segments 29 -> 34
Other:
- note added: "SSD1306 Header"
- moved on the sheet: J1
Changed lines of the file:
@@
 ESP32 Schematic
 Wire Wire Line
-	9150 1600 9000 1600
-Text GLabel 8800 1500 0    50   Input ~ 0
+	9900 1450 9750 1450
+Text GLabel 9550 1350 0    50   Input ~ 0
 SCL
-Text GLabel 9000 1600 0    50   Input ~ 0
+Text GLabel 9750 1450 0    50   Input ~ 0
 SDA
 $Comp
 L power:+3V3 #PWR04
 U 1 1 61B02C5C
-P 8450 1850
-F 0 "#PWR04" H 8450 1700 50  0001 C CNN
-F 1 "+3V3" H 8465 2023 50  0000 C CNN
-F 2 "" H 8450 1850 50  0001 C CNN
-F 3 "" H 8450 1850 50  0001 C CNN
-	1    8450 1850
-	-1   0    0    1
-$EndComp
-Text Notes 8350 2350 0    118  ~ 0
+P 9200 1700
+F 0 "#PWR04" H 9200 1550 50  0001 C CNN
+F 1 "+3V3" H 9215 1873 50  0000 C CNN
+F 2 "" H 9200 1700 50  0001 C CNN
+F 3 "" H 9200 1700 50  0001 C CNN
+	1    9200 1700
+	-1   0    0    1
+$EndComp
+Text Notes 9100 2200 0    118  ~ 0
 SCD-41 Header
 Wire Wire Line
@@
 	1250 1600 1500 1600
 Connection ~ 1500 1600
-Wire Wire Line
-	9700 3650 9700 3750
 $Comp
 L power:GND #PWR03
@@
 L Connector:Conn_01x04_Male J1
 U 1 1 6209986D
-P 9350 1700
-F 0 "J1" H 9458 1981 50  0000 C CNN
-F 1 "Conn_01x04_Male" H 9458 1890 50  0000 C CNN
-F 2 "Connector_PinSocket_2.54mm:PinSocket_1x04_P2.54mm_Vertical" H 9350 1700 50  0001 C CNN
-F 3 "~" H 9350 1700 50  0001 C CNN
-	1    9350 1700
+P 10100 1550
+F 0 "J1" H 10208 1831 50  0000 C CNN
+F 1 "Conn_01x04_Male" H 10208 1740 50  0000 C CNN
+F 2 "Connector_PinSocket_2.54mm:PinSocket_1x04_P2.54mm_Vertical" H 10100 1550 50  0001 C CNN
+F 3 "~" H 10100 1550 50  0001 C CNN
+	1    10100 1550
 	-1   0    0    1
 $EndComp
@@
 L power:GND #PWR05
 U 1 1 620A1AD1
-P 8600 1850
-F 0 "#PWR05" H 8600 1600 50  0001 C CNN
-F 1 "GND" H 8605 1677 50  0000 C CNN
-F 2 "" H 8600 1850 50  0001 C CNN
-F 3 "" H 8600 1850 50  0001 C CNN
-	1    8600 1850
-	1    0    0    -1
-$EndComp
-Wire Wire Line
-	8600 1800 8600 1850
-Wire Wire Line
-	8600 1800 9150 1800
-Wire Wire Line
-	8450 1850 8450 1700
-Wire Wire Line
-	8450 1700 9150 1700
-Wire Wire Line
-	8800 1500 9150 1500
-Wire Notes Line
-	8300 1400 9800 1400
-Wire Notes Line
-	9800 1400 9800 2400
-Wire Notes Line
-	9800 2400 8300 2400
-Wire Notes Line
-	8300 1400 8300 2400
+P 9350 1700
+F 0 "#PWR05" H 9350 1450 50  0001 C CNN
+F 1 "GND" H 9355 1527 50  0000 C CNN
+F 2 "" H 9350 1700 50  0001 C CNN
+F 3 "" H 9350 1700 50  0001 C CNN
+	1    9350 1700
+	1    0    0    -1
+$EndComp
+Wire Wire Line
+	9350 1650 9350 1700
+Wire Wire Line
+	9350 1650 9900 1650
+Wire Wire Line
+	9200 1700 9200 1550
+Wire Wire Line
+	9200 1550 9900 1550
+Wire Wire Line
+	9550 1350 9900 1350
+Wire Notes Line
+	9050 1250 10550 1250
+Wire Notes Line
+	10550 1250 10550 2250
+Wire Notes Line
+	10550 2250 9050 2250
+Wire Notes Line
+	9050 1250 9050 2250
 Wire Wire Line
 	1700 1850 950  1850
@@
 Wire Wire Line
 	9300 3250 9700 3250
-Wire Wire Line
-	9700 3250 9700 3350
-$Comp
-L Device:R_US R1
-U 1 1 624E061B
-P 9700 3500
-F 0 "R1" H 9768 3546 50  0000 L CNN
-F 1 "10k" H 9768 3455 50  0000 L CNN
-F 2 "SamacSys_Parts:RESC5025X70N" V 9740 3490 50  0001 C CNN
-F 3 "~" H 9700 3500 50  0001 C CNN
-	1    9700 3500
-	1    0    0    -1
-$EndComp
 Wire Notes Line
 	7900 2850 10000 2850
@@
 NoConn ~ 6350 1400
 NoConn ~ 6350 1500
+Wire Wire Line
+	9700 3250 9700 3750
+Wire Wire Line
+	8300 1450 8150 1450
+Text GLabel 7950 1350 0    50   Input ~ 0
+SCL
+Text GLabel 8150 1450 0    50   Input ~ 0
+SDA
+$Comp
+L power:+3V3 #PWR0101
+U 1 1 62500BEB
+P 7600 1700
+F 0 "#PWR0101" H 7600 1550 50  0001 C CNN
+F 1 "+3V3" H 7615 1873 50  0000 C CNN
+F 2 "" H 7600 1700 50  0001 C CNN
+F 3 "" H 7600 1700 50  0001 C CNN
+	1    7600 1700
+	-1   0    0    1
+$EndComp
+Text Notes 7500 2200 0    118  ~ 0
+SSD1306 Header
+$Comp
+L Connector:Conn_01x04_Male J3
+U 1 1 62500BF2
+P 8500 1550
+F 0 "J3" H 8608 1831 50  0000 C CNN
+F 1 "Conn_01x04_Male" H 8608 1740 50  0000 C CNN
+F 2 "Connector_PinSocket_2.54mm:PinSocket_1x04_P2.54mm_Vertical" H 8500 1550 50  0001 C CNN
+F 3 "~" H 8500 1550 50  0001 C CNN
+	1    8500 1550
+	-1   0    0    1
+$EndComp
+$Comp
+L power:GND #PWR0102
+U 1 1 62500BF8
+P 7750 1700
+F 0 "#PWR0102" H 7750 1450 50  0001 C CNN
+F 1 "GND" H 7755 1527 50  0000 C CNN
+F 2 "" H 7750 1700 50  0001 C CNN
+F 3 "" H 7750 1700 50  0001 C CNN
+	1    7750 1700
+	1    0    0    -1
+$EndComp
+Wire Wire Line
+	7750 1650 7750 1700
+Wire Wire Line
+	7750 1650 8300 1650
+Wire Wire Line
+	7600 1700 7600 1550
+Wire Wire Line
+	7600 1550 8300 1550
+Wire Wire Line
+	7950 1350 8300 1350
+Wire Notes Line
+	9000 1250 9000 2250
+Wire Notes Line
+	7450 1250 7450 2250
+Wire Notes Line
+	7450 1250 9000 1250
+Wire Notes Line
+	7450 2250 9000 2250
 $EndSCHEMATC
