File: UA-IOTENSR/UA-IOTENSR.kicad_pcb (KiCad board)
At the start: 4 copper layers, 80 x 79.1 mm, 38 parts, among them IC1 BQ2000TPN-B5, J1 Conn_01x04_Male, J2 ZX62-AB-5PA_31_, SW1 SW_Push, U1 ESP32-S3-MINI-1, U2 AP63203WU

Commit message: Zettai Ryouiki
Parts:
- removed R1: 10k, SamacSys_Parts:RESC5025X70N
- added J3: Conn_01x04_Male, Connector_PinSocket_2.54mm:PinSocket_1x04_P2.54mm_Vertical, F.Cu at (137.9, 90.2)
Connections:
- J2 pad 5: Net-(J2-Pad5) -> GNDREF
- J2 pad MP1: Net-(J2-Pad5) -> GNDREF
- J2 pad MP2: Net-(J2-Pad5) -> GNDREF
- J2 pad MP3: Net-(J2-Pad5) -> GNDREF
- J2 pad MP4: Net-(J2-Pad5) -> GNDREF
- J2 pad MP5: Net-(J2-Pad5) -> GNDREF
- J2 pad MP6: Net-(J2-Pad5) -> GNDREF
- SW1 pad 2: Net-(R1-Pad1) -> BAT-
Routing:
- net BAT-: track 12.9 -> 86.7 mm, vias 0 -> 5
- net DC+: track 0.00 -> 60.4 mm, vias 0 -> 2
- net +3V3: track 6.26 -> 63.5 mm
- net GNDREF: track 0.00 -> 52.8 mm, vias 0 -> 2
- net Net-(R8-Pad1): track 0.00 -> 46.1 mm
- net Net-(Cf1-Pad1): track 0.00 -> 24.0 mm, vias 0 -> 2
- net PUSHBUTTON: track 0.00 -> 19.4 mm
- net BAT+: track 5.01 -> 24.0 mm, vias 0 -> 3
- net SDA: track 0.00 -> 15.9 mm
- net Net-(Cmto1-Pad2): track 0.00 -> 14.5 mm, vias 0 -> 2
- net SCL: track 0.00 -> 13.1 mm
- net Net-(C1-Pad1): track 0.00 -> 11.0 mm
- net Net-(D2-Pad1): track 0.00 -> 9.92 mm, vias 0 -> 2
- net Net-(C5-Pad1): track 0.00 -> 7.45 mm
- net Net-(R4-Pad2): track 0.00 -> 7.38 mm
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- added copper zone on In2.Cu, net BAT+
Other:
- board text added: "SCD-41 HEADER"
- board text added: "SSD1306 HEADER"
- board text removed: "I2C CONN"
